File: nrf52840_pmw3360.kicad_sch (KiCad schematic)
At the start: 2 parts, among them J1 PMW3360_Breakout, U1 SuperMini_nRF52840

Commit message: feat: J2バッテリーコネクタ追加（B+→BATIN/P0.04、B-→GND）
Parts:
- added J2: Battery_JST-PH_2pin, Connector_JST:JST_PH_B2B-PH-K_1x02_P2.00mm_Vertical, symbol Battery_Connector_2pin
Connections:
- net GND: now also J2.2 (B-)
- net BATIN: now reaches U1.24 (BATIN/P0.04)
- net BATIN: now also J2.1 (B+)
- no-connect marks 16 -> 15
Changed lines of the file:
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@@
     (comment 2 "PMW3360 Breakout Board (monkeypad/pmw3360-breakout)")
     (comment 3 "SPI: MOSI=P0.10  MISO=P1.11  SCK=P1.13  NCS=P1.06")
-    (comment 4 "MOTION=P1.04  VCC=3.3V from SuperMini pin21")
+    (comment 4 "MOTION=P1.04  VCC=3.3V from SuperMini pin21  BAT+=BATIN/P0.04")
   )
   (symbol (lib_id "SuperMini_nRF52840") (at 100.0000 100.0000 0) (unit 1)
@@
       (effects (font (size 1.27 1.27))))
     (property "Footprint" "Connector_PinHeader_2.54mm:PinHeader_1x08_P2.54mm_Vertical" (at 162.0000 107.0000 0)
+      (effects (font (size 1.27 1.27)) (hide yes)))
+  )
+  (symbol (lib_id "Battery_Connector_2pin") (at 130.0000 135.0000 0) (unit 1)
+    (in_bom yes) (on_board yes) (dnp no)
+    (property "Reference" "J2" (at 130.0000 130.4600 0)
+      (effects (font (size 1.27 1.27))))
+    (property "Value" "Battery_JST-PH_2pin" (at 130.0000 139.0400 0)
+      (effects (font (size 1.27 1.27))))
+    (property "Footprint" "Connector_JST:JST_PH_B2B-PH-K_1x02_P2.00mm_Vertical" (at 130.0000 135.0000 0)
       (effects (font (size 1.27 1.27)) (hide yes)))
   )
@@
     (effects (font (size 1.27 1.27)))
 )
+  (wire (pts (xy 116.0300 133.7300) (xy 121.1100 133.7300))
+    (stroke (width 0) (type default))
+)
+  (label "BATIN" (at 116.0300 133.7300 180)
+    (effects (font (size 1.27 1.27)))
+)
+  (symbol (lib_id "power:GND") (at 118.5700 136.2700 0) (unit 1)
+    (in_bom yes) (on_board yes) (dnp no)
+    (property "Reference" "#PWR07" (at 118.5700 136.2700 0)
+      (effects (font (size 1.27 1.27)) (hide yes)))
+    (property "Value" "GND" (at 118.5700 136.2700 0)
+      (effects (font (size 1.27 1.27))))
+  )
+  (wire (pts (xy 118.5700 136.2700) (xy 121.1100 136.2700))
+    (stroke (width 0) (type default))
+)
+  (wire (pts (xy 110.1600 113.9700) (xy 115.2400 113.9700))
+    (stroke (width 0) (type default))
+)
+  (label "BATIN" (at 115.2400 113.9700 0)
+    (effects (font (size 1.27 1.27)))
+)
   (no_connect (at 89.8400 86.0300))
   (no_connect (at 89.8400 88.5700))
@@
   (no_connect (at 110.1600 103.8100))
   (no_connect (at 110.1600 108.8900))
-  (no_connect (at 110.1600 113.9700))
   (no_connect (at 153.1100 103.1900))
 )
