File: nrf52840_pmw3360.kicad_pcb (KiCad board)
At the start: 2 copper layers, 18 x 33 mm, 3 parts, among them J1 PMW3360_Breakout, J2 Battery_JST-PH, U1 SuperMini_nRF52840

Commit message: fix: KiCad 9.0対応 F.CrtYdレイヤー番号修正・stroke形式対応
Other:
- rule pad_to_mask_clearance: 0.05 -> 0
Changed lines of the file:
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@@
-(kicad_pcb (version 20221018) (generator pcbnew)
-  (general (thickness 1.6) (legacy_teardrops no))
+(kicad_pcb (version 20240108) (generator pcbnew) (generator_version "9.0")
+  (general (thickness 1.6))
   (paper "A4")
   (title_block
@@
     (0 "F.Cu" signal)
     (31 "B.Cu" signal)
+    (34 "B.Paste" user)
     (35 "F.Paste" user)
-    (36 "F.SilkS" user "F.Silkscreen")
-    (37 "B.SilkS" user "B.Silkscreen")
-    (38 "F.Mask" user)
-    (39 "B.Mask" user)
+    (36 "B.SilkS" user)
+    (37 "F.SilkS" user)
+    (38 "B.Mask" user)
+    (39 "F.Mask" user)
     (44 "Edge.Cuts" user)
     (45 "Margin" user)
-    (50 "F.Courtyard" user)
-    (51 "B.Courtyard" user)
-    (52 "F.Fab" user)
-    (53 "B.Fab" user)
+    (46 "B.CrtYd" user)
+    (47 "F.CrtYd" user)
+    (48 "B.Fab" user)
+    (49 "F.Fab" user)
   )
   (setup
-    (pad_to_mask_clearance 0.05)
+    (pad_to_mask_clearance 0)
     (allow_soldermask_bridges_in_footprints no)
     (pcbplotparams
@@
       (plotreference yes)
       (plotvalue yes)
-      (plotfptext yes)
       (plotinvisibletext no)
       (sketchpadsonfab no)
@@
   (net 7 "MOTION")
   (net 8 "BATIN")
-  (gr_rect (start 0 0) (end 18.0000 33.0000) (layer "Edge.Cuts") (width 0.05))
-  (gr_line (start 0.00 0.00) (end 1.00 0.00) (layer "F.SilkS") (width 0.12))
-  (gr_line (start 0.00 0.00) (end 0.00 1.00) (layer "F.SilkS") (width 0.12))
-  (gr_line (start 18.00 0.00) (end 17.00 0.00) (layer "F.SilkS") (width 0.12))
-  (gr_line (start 18.00 0.00) (end 18.00 1.00) (layer "F.SilkS") (width 0.12))
-  (gr_line (start 18.00 33.00) (end 17.00 33.00) (layer "F.SilkS") (width 0.12))
-  (gr_line (start 18.00 33.00) (end 18.00 32.00) (layer "F.SilkS") (width 0.12))
-  (gr_line (start 0.00 33.00) (end 1.00 33.00) (layer "F.SilkS") (width 0.12))
-  (gr_line (start 0.00 33.00) (end 0.00 32.00) (layer "F.SilkS") (width 0.12))
+  (gr_rect (start 0 0) (end 18.0000 33.0000) (stroke (width 0.05) (type default)) (layer "Edge.Cuts"))
+  (gr_line (start 0.00 0.00) (end 1.00 0.00) (stroke (width 0.12) (type default)) (layer "F.SilkS"))
+  (gr_line (start 0.00 0.00) (end 0.00 1.00) (stroke (width 0.12) (type default)) (layer "F.SilkS"))
+  (gr_line (start 18.00 0.00) (end 17.00 0.00) (stroke (width 0.12) (type default)) (layer "F.SilkS"))
+  (gr_line (start 18.00 0.00) (end 18.00 1.00) (stroke (width 0.12) (type default)) (layer "F.SilkS"))
+  (gr_line (start 18.00 33.00) (end 17.00 33.00) (stroke (width 0.12) (type default)) (layer "F.SilkS"))
+  (gr_line (start 18.00 33.00) (end 18.00 32.00) (stroke (width 0.12) (type default)) (layer "F.SilkS"))
+  (gr_line (start 0.00 33.00) (end 1.00 33.00) (stroke (width 0.12) (type default)) (layer "F.SilkS"))
+  (gr_line (start 0.00 33.00) (end 0.00 32.00) (stroke (width 0.12) (type default)) (layer "F.SilkS"))
 (footprint "SuperMini_nRF52840_Socket" (layer "F.Cu") (at 0 0)
   (fp_text reference "U1" (at 5.0000 1.3100) (layer "F.SilkS")
@@
     (pad "23" thru_hole circle (at 16.7300 29.2100) (size 1.6000 1.6000) (drill 1.0000) (layers "*.Cu" "*.Mask") (net 1 "GND"))
     (pad "24" thru_hole circle (at 16.7300 31.7500) (size 1.6000 1.6000) (drill 1.0000) (layers "*.Cu" "*.Mask") (net 8 "BATIN"))
-  (fp_line (start -0.2300 2.3100) (end 18.2300 2.3100) (layer "F.SilkS") (width 0.1200))
-  (fp_line (start 18.2300 2.3100) (end 18.2300 33.2500) (layer "F.SilkS") (width 0.1200))
-  (fp_line (start 18.2300 33.2500) (end -0.2300 33.2500) (layer "F.SilkS") (width 0.1200))
-  (fp_line (start -0.2300 33.2500) (end -0.2300 2.3100) (layer "F.SilkS") (width 0.1200))
+  (fp_line (start -0.2300 2.3100) (end 18.2300 2.3100) (stroke (width 0.1200) (type default)) (layer "F.SilkS"))
+  (fp_line (start 18.2300 2.3100) (end 18.2300 33.2500) (stroke (width 0.1200) (type default)) (layer "F.SilkS"))
+  (fp_line (start 18.2300 33.2500) (end -0.2300 33.2500) (stroke (width 0.1200) (type default)) (layer "F.SilkS"))
+  (fp_line (start -0.2300 33.2500) (end -0.2300 2.3100) (stroke (width 0.1200) (type default)) (layer "F.SilkS"))
+  (fp_line (start -0.4800 2.0600) (end 18.4800 2.0600) (stroke (width 0.0500) (type default)) (layer "F.CrtYd"))
+  (fp_line (start 18.4800 2.0600) (end 18.4800 33.5000) (stroke (width 0.0500) (type default)) (layer "F.CrtYd"))
+  (fp_line (start 18.4800 33.5000) (end -0.4800 33.5000) (stroke (width 0.0500) (type default)) (layer "F.CrtYd"))
+  (fp_line (start -0.4800 33.5000) (end -0.4800 2.0600) (stroke (width 0.0500) (type default)) (layer "F.CrtYd"))
   (fp_text user "1" (at 0.2700 3.8100) (layer "F.SilkS")
     (effects (font (size 0.6 0.6) (thickness 0.15))))
@@
     (pad "7" thru_hole circle (at 15.3500 1.2700) (size 1.6000 1.6000) (drill 1.0000) (layers "*.Cu" "*.Mask") (net 4 "MISO"))
     (pad "8" thru_hole circle (at 17.8900 1.2700) (size 1.6000 1.6000) (drill 1.0000) (layers "*.Cu" "*.Mask") (net 6 "NCS"))
-  (fp_line (start -1.1900 -0.0300) (end 19.1900 -0.0300) (layer "F.SilkS") (width 0.1200))
-  (fp_line (start 19.1900 -0.0300) (end 19.1900 2.5700) (layer "F.SilkS") (width 0.1200))
-  (fp_line (start 19.1900 2.5700) (end -1.1900 2.5700) (layer "F.SilkS") (width 0.1200))
-  (fp_line (start -1.1900 2.5700) (end -1.1900 -0.0300) (layer "F.SilkS") (width 0.1200))
+  (fp_line (start -1.1900 -0.0300) (end 19.1900 -0.0300) (stroke (width 0.1200) (type default)) (layer "F.SilkS"))
+  (fp_line (start 19.1900 -0.0300) (end 19.1900 2.5700) (stroke (width 0.1200) (type default)) (layer "F.SilkS"))
+  (fp_line (start 19.1900 2.5700) (end -1.1900 2.5700) (stroke (width 0.1200) (type default)) (layer "F.SilkS"))
+  (fp_line (start -1.1900 2.5700) (end -1.1900 -0.0300) (stroke (width 0.1200) (type default)) (layer "F.SilkS"))
+  (fp_line (start -1.4400 -0.2800) (end 19.4400 -0.2800) (stroke (width 0.0500) (type default)) (layer "F.CrtYd"))
+  (fp_line (start 19.4400 -0.2800) (end 19.4400 2.8200) (stroke (width 0.0500) (type default)) (layer "F.CrtYd"))
+  (fp_line (start 19.4400 2.8200) (end -1.4400 2.8200) (stroke (width 0.0500) (type default)) (layer "F.CrtYd"))
+  (fp_line (start -1.4400 2.8200) (end -1.4400 -0.2800) (stroke (width 0.0500) (type default)) (layer "F.CrtYd"))
   (fp_text user "GND" (at 0.1100 3.2700) (layer "F.SilkS")
     (effects (font (size 0.5 0.5) (thickness 0.15))))
@@
     (pad "1" thru_hole oval (at 8.0000 20.0000) (size 1.6000 1.6000) (drill 0.8000) (layers "*.Cu" "*.Mask") (net 8 "BATIN"))
     (pad "2" thru_hole circle (at 10.0000 20.0000) (size 1.6000 1.6000) (drill 0.8000) (layers "*.Cu" "*.Mask") (net 1 "GND"))
-  (fp_line (start 6.8000 18.8000) (end 11.2000 18.8000) (layer "F.SilkS") (width 0.1200))
-  (fp_line (start 11.2000 18.8000) (end 11.2000 21.2000) (layer "F.SilkS") (width 0.1200))
-  (fp_line (start 11.2000 21.2000) (end 6.8000 21.2000) (layer "F.SilkS") (width 0.1200))
-  (fp_line (start 6.8000 21.2000) (end 6.8000 18.8000) (layer "F.SilkS") (width 0.1200))
+  (fp_line (start 6.5500 18.5500) (end 11.4500 18.5500) (stroke (width 0.0500) (type default)) (layer "F.CrtYd"))
+  (fp_line (start 11.4500 18.5500) (end 11.4500 21.4500) (stroke (width 0.0500) (type default)) (layer "F.CrtYd"))
+  (fp_line (start 11.4500 21.4500) (end 6.5500 21.4500) (stroke (width 0.0500) (type default)) (layer "F.CrtYd"))
+  (fp_line (start 6.5500 21.4500) (end 6.5500 18.5500) (stroke (width 0.0500) (type default)) (layer "F.CrtYd"))
+  (fp_line (start 6.8000 18.8000) (end 11.2000 18.8000) (stroke (width 0.1200) (type default)) (layer "F.SilkS"))
+  (fp_line (start 11.2000 18.8000) (end 11.2000 21.2000) (stroke (width 0.1200) (type default)) (layer "F.SilkS"))
+  (fp_line (start 11.2000 21.2000) (end 6.8000 21.2000) (stroke (width 0.1200) (type default)) (layer "F.SilkS"))
+  (fp_line (start 6.8000 21.2000) (end 6.8000 18.8000) (stroke (width 0.1200) (type default)) (layer "F.SilkS"))
   (fp_text user "B+" (at 8.0000 18.0000) (layer "F.SilkS")
     (effects (font (size 0.6 0.6) (thickness 0.15))))
